Commit message: 0805_update

File: 基础环境检查/deploy_eva_robot检测/robot/g1_description/g1_29dof_mode_15_with_dex1_1.urdf (robot description, URDF)
Before this commit: robot g1_29dof_mode_15, 43 links, 42 joints
Joints:
- removed joint left_gripper_joint
- removed joint left_gripper_mimic_joint
- removed joint right_gripper_joint
- removed joint right_gripper_mimic_joint
- added joint left_dex1_finger_joint_1: type prismatic, parent left_dex1_base_link, child left_dex1_finger_link_1, origin xyz=0 0 0 rpy=0 0 0, axis 0 -1 0, limit lower=-0.02 upper=0.0245 effort=20 velocity=0.2
- added joint left_dex1_finger_joint_2: type prismatic, parent left_dex1_base_link, child left_dex1_finger_link_2, origin xyz=0 0 0 rpy=0 0 0, axis 0 1 0, limit lower=-0.02 upper=0.0245 effort=20 velocity=0.2, mimic joint=left_dex1_finger_joint_1 multiplier=1 offset=0
- added joint right_dex1_finger_joint_1: type prismatic, parent right_dex1_base_link, child right_dex1_finger_link_1, origin xyz=0 0 0 rpy=0 0 0, axis 0 -1 0, limit lower=-0.02 upper=0.0245 effort=20 velocity=0.2
- added joint right_dex1_finger_joint_2: type prismatic, parent right_dex1_base_link, child right_dex1_finger_link_2, origin xyz=0 0 0 rpy=0 0 0, axis 0 1 0, limit lower=-0.02 upper=0.0245 effort=20 velocity=0.2, mimic joint=right_dex1_finger_joint_1 multiplier=1 offset=0
